Commit message: add LQR balancing controller and raise arm velocity limit
Derive the linearised model of the reaction wheel pendulum about upright from
the URDF inertias and solve for LQR gains.

State is x = [theta_base, omega_base, omega_arm]; theta_arm does not enter the
dynamics because the arm COM sits on its own pivot axis. Input is the torque on
body_arm. The base equation carries no torque term: the motor reaches the body
only through the inertial coupling I_a*theta_ddot_arm, which is the reaction
torque rewritten.

  I_b = (1/3) m_b L^2 + m_a L^2 = 1.8e-3
  I_a = 1.9e-5
  mgl = m_b g l_b + m_a g L = 0.0736   (matches the effort Isaac reports)

Q from Bryson's rule with budgets 0.785 rad, pi rad/s, 5 rad/s; R = 1e6.
Closed-loop poles -212.8 and -6.36 +/- 0.04j. The slow pole barely moves with R
because the open-loop instability at +6.4 rad/s sets a floor on recovery speed.

Raise the body_arm velocity limit from 10 to 100 rad/s. Integrating the base
equation over a recovery gives I_a*delta_omega_arm = mgl * integral(theta_base),
so the arm speed needed is mgl*theta_0*tau_c/I_a, about 61 rad/s from a 0.1 rad
disturbance. The old 10 rad/s limit made the problem infeasible at any gain, and
the arm saturating removes all control authority because a pinned arm produces no
reaction torque. Region of attraction is now theta_base < ~0.16 rad.

Add a staleness guard: if /joint_states is older than max_age, publish zero
effort rather than returning. Isaac holds the last command forever, so going
quiet would leave the last torque applied.

Stage changes: physxJoint:maxJointVelocity on body_arm (authored in degrees/s by
the URDF importer, so 5730), and the physics and timeline rates raised from 60.

File: urdf/body.urdf (robot description, URDF)
Before this commit: robot pendulum, 3 links, 2 joints
Joints:
- joint body_arm: limit effort=10.0 velocity=10.0 -> effort=10.0 velocity=100.0
